File: Electronic Throttle Controller/Hardware/Electronic Throttle Controller.kicad_sch (KiCad schematic)
At the start: 45 parts, among them J1 USB_B, J2 ETC SIG, J3 ETC CAN, J4 ETC PWR, Q1 ECH8697R, Q2 2N7002, U1 ESP32-C3-WROOM-02U, U2 MCP2551-I-SN, U3 AMS1117-3.3, U4 L7805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

Commit message: feat: change to stm32 and add IOC
Parts:
- removed C7, C8, C9: 100nF, Capacitor_SMD:C_0603_1608Metric, symbol Device:C
- removed J1: USB_B, Connector_USB:USB_B_TE_5787834_Vertical, symbol Connector:USB_B
- removed Q1: ECH8697R, Package_TO_SOT_SMD:OnSemi_ECH8, symbol Device:Q_Dual_NMOS_S1G1S2G2D2D2D1D1
- removed R13, R14: 4.7K, Resistor_SMD:R_0603_1608Metric, symbol Device:R
- removed R15, R16, R17: 10K, Resistor_SMD:R_0603_1608Metric, symbol Device:R
- removed U1: ESP32-C3-WROOM-02U, RF_Module:ESP32-C3-WROOM-02U, symbol RF_Module:ESP32-C3-WROOM-02U
- removed U5, U6, U7: ADS1115IDGS, Package_SO:TSSOP-10_3x3mm_P0.5mm, symbol Analog_ADC:ADS1115IDGS
- added D2: 1N47xxA, Diode_THT:D_DO-41_SOD81_P10.16mm_Horizontal, symbol Diode:1N47xxA
- added Q1, Q3, Q4, Q5: AO3400A, Package_TO_SOT_SMD:SOT-23, symbol Transistor_FET:AO3400A
- added Q6, Q7: 2N7002, Package_TO_SOT_SMD:SOT-23, symbol Transistor_FET:2N7002
- added R21: 10K, Resistor_SMD:R_0603_1608Metric, symbol Device:R
- added R22: 100, Resistor_SMD:R_0603_1608Metric, symbol Device:R
- added TH1, TH2: 10K, Resistor_SMD:R_0603_1608Metric, symbol Device:Thermistor
- added U1: ACS722xLCTR-20AU, Package_SO:SOIC-8_3.9x4.9mm_P1.27mm, symbol Sensor_Current:ACS722xLCTR-20AU
- added U8: STM32F042K6Tx, Package_QFP:LQFP-32_7x7mm_P0.8mm, symbol MCU_ST_STM32F0:STM32F042K6Tx
- added U9: AMS1117-3.3, Package_TO_SOT_SMD:SOT-223-3_TabPin2, symbol Regulator_Linear:AMS1117-3.3
- R3: value 100 -> 10K
- R4: value 10K -> 100
Connections:
- net +3.3V: now also R3.2, R21.2, U8.1 (VDD), U8.17 (VDDIO2)
- net +5V: now also R5.2
- net +5VA: now also U9.3 (VI)
- net -BATT: now also Q1.2 (S), Q3.2 (S), Q4.2 (S), Q5.2 (S), Q6.2 (S), Q7.2 (S), U8.16 (VSS), U9.1 (GND); no longer R4.1, R5.1
- net APPS1_SIGF: now also U8.6 (PA0)
- net APPS2_SIGF: now also U8.7 (PA1)
- net BLIP_SIG: now also R4.1; no longer R4.2
- net BPTF_SIGF: now also U8.8 (PA2)
- net BPTR_SIGF: now also U8.9 (PA3)
- net CAN_RX: now also U8.21 (PA11)
- net CAN_TX: now also U8.22 (PA12)
- net GNDA: now also U8.32 (VSSA)
- net MOTOR_CTRL: now also R21.1, R22.1; no longer R5.2, R6.1
- net MOTOR_GND: now also Q1.3 (D), Q3.3 (D), Q4.3 (D), Q5.3 (D)
- net TPS1_SIGF: now also U8.10 (PA4)
- net TPS2_SIGF: now also U8.11 (PA5)
- net ETB_DRIVER_GATE: now reaches R6.2
- net ETB_DRIVER_GATE: now also Q1.1 (G), Q3.1 (G), Q4.1 (G), Q5.1 (G)
- new net: Q6.1 (G), R22.2
- new net: Q6.3 (D), Q7.3 (D), R5.1, R6.1
- new net: U1.1 (IP+), U1.2 (IP+)
- new net: U1.3 (IP-), U1.4 (IP-)
- new net: Q7.1 (G), R4.2
- new net +3.3VA: U8.5 (VDDA), U9.2 (VO)
- no-connect marks 9 -> 1
Other:
- note added: "STM32"
- note removed: "ESP32 + I2C Pullups"
- moved on the sheet: C1, C2, C3, C4, C5, C6, R10, R11, R12, R7, R8, R9
