File: BSPD/BSPD.kicad_sch (KiCad schematic)
At the start: 72 parts, among them J1 Signal, J2 Power, Q1 2N7002, Q2 BSS84, Q3 2N7002, Q4 2N7002, Q5 2N7002, Q6 2N7002, U1 LM339, U2 LM339

Commit message: docs: document bspd rev A errata and update schematic
Parts:
- removed R10: 10K, Resistor_SMD:R_0603_1608Metric, symbol Device:R
- added R3: 10K, Resistor_SMD:R_0603_1608Metric, symbol Device:R
- TP1: value TPS OV -> TPS UV
- TP2: value TPS UV -> TPS OV
- TP3: value BPT OV -> BPT UV
- TP4: value BPT UV -> BPT OV
- TP9: value ~{PANIC BRAKE} -> PANIC BRAKE
Connections:
- net 1_RC: now also U1.8 (-); no longer U1.9 (+)
- net SENSORS_OK: now also R3.1
- net ~{PANIC_BRAKE}: no longer D1.2 (A), R11.1, R24.1, TP9.1, U1.1, U1.2
- net at C4.1, R11.2, TP15.1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: now also D1.2 (A); no longer D1.1 (K)
- net at C3.1, D4.1 (K), TP16.1: now also U1.9 (+), R3.2; no longer U1.8 (-)
- net at C5.1, R19.1, TP13.1: now also Q2.2 (S); no longer Q2.3 (D)
- net at R18.2, R25.2: now also Q2.3 (D); no longer Q2.2 (S)
- new net PANIC_BRAKE: D1.1 (K), R11.1, R24.1, TP9.1, U1.1, U1.2
Other:
- moved on the sheet: D1

Commit message: feat: begin rev b
- Change parts to reduce cost (remove extended components)
- Reset PCB to prep layout
- Switch to resistor dividers
Parts:
- removed D1, D4: BAT43W-V, Diode_SMD:D_SOD-123, symbol Diode:BAT43W-V
- removed D2, D3: ESDA-05N, Diode_SMD:D_0603_1608Metric, symbol Diode:ESD9B5.0ST5G
- removed H1: MountingHole, MountingHole:MountingHole_3.2mm_M3, symbol Mechanical:MountingHole
- removed Q2: BSS84, Package_TO_SOT_SMD:SOT-23, symbol Transistor_FET:BSS84
- removed RV1, RV2, RV3, RV4, RV5, RV6: 3314J-1-103E, Potentiometer_SMD:Potentiometer_Bourns_3314J_Vertical, symbol Device:R_Potentiometer_Trim
- removed TP1: TPS UV, TestPoint:TestPoint_Keystone_5005-5009_Compact, symbol Connector:TestPoint
- removed TP13: Latching RC, TestPoint:TestPoint_Keystone_5005-5009_Compact, symbol Connector:TestPoint
- removed TP15: ~{PANIC BRAKE} RC, TestPoint:TestPoint_Keystone_5005-5009_Compact, symbol Connector:TestPoint
- removed TP16: SENSORS_OK RC, TestPoint:TestPoint_Keystone_5005-5009_Compact, symbol Connector:TestPoint
- removed TP2: TPS OV, TestPoint:TestPoint_Keystone_5005-5009_Compact, symbol Connector:TestPoint
- removed TP3: BPT UV, TestPoint:TestPoint_Keystone_5005-5009_Compact, symbol Connector:TestPoint
- removed TP4: BPT OV, TestPoint:TestPoint_Keystone_5005-5009_Compact, symbol Connector:TestPoint
- removed TP5: TPS 10%, TestPoint:TestPoint_Keystone_5005-5009_Compact, symbol Connector:TestPoint
- removed TP6: BPT HB, TestPoint:TestPoint_Keystone_5005-5009_Compact, symbol Connector:TestPoint
- removed TP7: TAU, TestPoint:TestPoint_Keystone_5005-5009_Compact, symbol Connector:TestPoint
- added D1, D4: RB160M-30, Diode_SMD:D_SOD-123, symbol Device:D_Schottky
- added D2, D3: SMAJ5.0A, Diode_SMD:D_SMA, symbol Diode:SMAJ5.0A
- added H1: MountingHole_Pad, MountingHole:MountingHole_3.2mm_M3_DIN965_Pad, symbol Mechanical:MountingHole_Pad
- added Q2: AO3401A, Package_TO_SOT_SMD:SOT-23, symbol Transistor_FET:AO3401A
- added R10, R20, R21, R22, R23, R4, R5, R6, R8, R9: 100K, Resistor_SMD:R_0603_1608Metric, symbol Device:R
- C1, C2: value 150nF -> 220nF
Connections:
- net +5VA: now also R20.1, R22.1, R5.1, R8.1
- net BPT_SIG: now also D2.1 (A1)
- net GNDA: now also D2.2 (A2), D3.2 (A2), R10.2, R21.2, R23.2, R6.2
- net PANIC_BRAKE: now also D1.1 (K)
- net SENSORS_OK: now also D4.2 (A)
- net TPS_SIG: now also D3.1 (A1)
- net at U1.4 (-): now also R20.2, R21.1
- net at C4.1, R11.2, U1.10 (-): now also D1.2 (A)
- net at U1.6 (-): now also R22.2, R23.1
- net at C3.1, R3.2, U1.9 (+): now also D4.1 (K)
- net at U2.8 (-): now also R4.2, R6.1
- net at U2.11 (+): now also R4.1, R5.2
- net at C5.1, R19.1: now also Q2.2 (S)
- net at R18.2, R25.2: now also Q2.3 (D)
- net at R17.2: now also Q2.1 (G)
- net at U2.7 (+): now also R8.2, R9.1
- net at U2.4 (-): now also R10.1, R9.2
- no-connect marks 0 -> 1
Other:
- note added: "Signal Pulldown, ESD Protection & Low Pass Filter (-3dB = ~72Hz)"
- note removed: "Signal Pulldown, ESD Protection & Low Pass Filter (-3dB = ~106Hz)"
- moved on the sheet: C1, C2, R14, R15, R2, TP9

Commit message: feat: add onboard regulator to reduce startup requirements
(not set in stone)
Parts:
- removed Q1, Q6: 2N7002, Package_TO_SOT_SMD:SOT-23, symbol Transistor_FET:2N7002
- removed R22, R23: 100K, Resistor_SMD:R_0603_1608Metric, symbol Device:R
- added C10, C12: 10uF, Capacitor_SMD:C_0603_1608Metric, symbol Device:C
- added C11, C13: 100nF, Capacitor_SMD:C_0603_1608Metric, symbol Device:C
- added Q1, Q6: AO3400A, Package_TO_SOT_SMD:SOT-23, symbol Transistor_FET:AO3400A
- added U3: HT7533-1-SOT89, Package_TO_SOT_SMD:SOT-89-3, symbol Regulator_Linear:HT75xx-1-SOT89
Connections:
- net +5VA: no longer R16.2, R19.2, R20.1, R24.2, R7.2
- net +BATT: now also C12.1, C13.1, U3.2 (VIN)
- net -BATT: now also C10.2, C11.2, C12.2, C13.2, Q6.2 (S), U3.1 (GND)
- net BSPD_OK: now also Q1.3 (D), Q6.1 (G)
- net BSPD_SD-: now also Q6.3 (D)
- net GNDA: now also Q1.2 (S); no longer R21.2
- net BPT_HB_TH: now reaches U1.6 (-)
- net BPT_HB_TH: now also R20.2, R9.1
- net TPS_HB_TH: now reaches R21.1, U1.4 (-)
- net TPS_HB_TH: now also R4.2; no longer R20.2
- net at R6.1, U2.8 (-): now also R21.2; no longer R4.2
- net at R18.1: now also Q1.1 (G)
- net at R8.2, U2.7 (+): now also R20.1; no longer R9.1
- new net +3.3V: C10.1, C11.1, R16.2, R19.2, R24.2, R7.2, U3.3 (VOUT)
Other:
- moved on the sheet: R10, R4, R5, R6, R8, R9, U1A

Commit message: BSPD rev 2a
Parts:
- removed C12: 10uF, Capacitor_SMD:C_0603_1608Metric, symbol Device:C
- removed C13: 100nF, Capacitor_SMD:C_0603_1608Metric, symbol Device:C
- removed D2, D3: SMAJ5.0A, Diode_SMD:D_SMA, symbol Diode:SMAJ5.0A
- removed D5, D6, D7, D8: LED, LED_SMD:LED_0603_1608Metric, symbol Device:LED
- removed H1: MountingHole_Pad, MountingHole:MountingHole_3.2mm_M3_DIN965_Pad, symbol Mechanical:MountingHole_Pad
- removed J1: Signal, Connector_PinHeader_2.54mm:PinHeader_1x04_P2.54mm_Vertical, symbol Connector_Generic:Conn_01x04
- removed J2: Power, Connector_PinHeader_2.54mm:PinHeader_1x03_P2.54mm_Vertical, symbol Connector_Generic:Conn_01x03
- removed Q3, Q4, Q5: 2N7002, Package_TO_SOT_SMD:SOT-23, symbol Transistor_FET:2N7002
- removed R10, R20, R21, R5, R6, R8, R9: 100K, Resistor_SMD:R_0603_1608Metric, symbol Device:R
- removed R26, R27, R30, R32: 4.7K, Resistor_SMD:R_0603_1608Metric, symbol Device:R
- removed R28, R29, R31: 10K, Resistor_SMD:R_0603_1608Metric, symbol Device:R
- removed TP10: GNDA, TestPoint:TestPoint_Keystone_5005-5009_Compact, symbol Connector:TestPoint
- removed TP11: BPT, TestPoint:TestPoint_Keystone_5005-5009_Compact, symbol Connector:TestPoint
- removed TP12: TPS, TestPoint:TestPoint_Keystone_5005-5009_Compact, symbol Connector:TestPoint
- removed TP14: BSPD OK, TestPoint:TestPoint_Keystone_5005-5009_Compact, symbol Connector:TestPoint
- removed TP8: SENSORS OK, TestPoint:TestPoint_Keystone_5005-5009_Compact, symbol Connector:TestPoint
- removed TP9: PANIC BRAKE, TestPoint:TestPoint_Keystone_5005-5009_Compact, symbol Connector:TestPoint
- removed U3: HT7533-1-SOT89, Package_TO_SOT_SMD:SOT-89-3, symbol Regulator_Linear:HT75xx-1-SOT89
- added D5: SM05, Package_TO_SOT_SMD:SOT-23, symbol Diode:BAT54A
- added J1: +BATT, RRM:PinHeader_1x01_P2.54mm_Vertical, symbol Connector_Generic:Conn_01x01
- added J10, J11, J12, J13, J14, J2, J3, J4, J5, J6, J7, J8, J9: +BATT, RRM:PinHeader_1x01_P2.54mm_Circular, symbol Connector_Generic:Conn_01x01
- R17, R18: value 10K -> 100
- R4: value 100K -> 100
- U1, U2: footprint Package_SO:SOIC-14_3.9x8.7mm_P1.27mm -> Package_DFN_QFN:WQFN-16-1EP_3x3mm_P0.5mm_EP1.75x1.75mm
Connections:
- net +3.3V is gone; now on net +5VA: C10.1, C11.1, R16.2, R19.2, R24.2, R7.2
- net +5VA: now also J11.1 (Pin_1)
- net +BATT: now also U1.1 (V+), U2.1 (V+), J1.1 (Pin_1); no longer U1.3 (V+), U2.3 (V+)
- net -BATT: now also Q1.2 (S), R25.1, U1.17 (Thermal), U2.17 (Thermal), J4.1 (Pin_1); no longer C10.2, C11.2
- net 1_RC: now also U1.8 (+), U1.9 (-); no longer U1.11 (+), U1.8 (-)
- net BPT: now also U1.4 (+), U2.4 (+), U2.5 (-); no longer U1.7 (+), U2.5 (+), U2.6 (-)
- net BPT_HB_TH: now also U1.2 (-), J6.1 (Pin_1); no longer U1.6 (-)
- net BPT_SIG: now also D5.1, J9.1 (Pin_1)
- net BSPD_OK: now also R4.1, U1.13, U1.14; no longer Q6.1 (G), U1.13, U1.14
- net BSPD_SD-: now also J2.1 (Pin_1)
- net GNDA: now also C10.2, C11.2, D5.3, J8.1 (Pin_1); no longer Q1.2 (S), R25.1
- net PANIC_BRAKE: now also U1.15, U1.16; no longer U1.1, U1.2
- net SENSORS_OK: now also U2.13, U2.14, U2.15, U2.16; no longer U2.1, U2.13, U2.14, U2.2
- net TPS: now also U1.6 (+), U2.8 (+); no longer U1.5 (+), U2.10 (-)
- net TPS_HB_TH: now also U1.5 (-), J13.1 (Pin_1); no longer R4.2, U1.4 (-)
- net TPS_SIG: now also D5.2, J10.1 (Pin_1)
- net BSPD_RST: now reaches Q2.3 (D), R18.2, R25.2
- net BSPD_RST: now also J3.1 (Pin_1)
- net at C4.1, D1.2 (A), R11.2: now also U1.7 (-); no longer U1.10 (-)
- net at C3.1, D4.1 (K), R3.2: now also U1.11 (+); no longer U1.9 (+)
- new net: Q6.1 (G), R4.2
- new net BPT_MAX_TH: J5.1 (Pin_1), U2.6 (+)
- new net BPT_MIN_TH: J7.1 (Pin_1), U2.2 (-)
- new net TPS_MAX_TH: J14.1 (Pin_1), U2.11 (+)
- new net TPS_MIN_TH: J12.1 (Pin_1), U2.7 (-)
- no-connect marks 1 -> 0
Other:
- note added: "BPT >HB Threshold (in volts)"
- note added: "SDC Driver"
- note added: "TPS >10% (in volts)"
- note removed: "BPT >1.8V"
- note removed: "Display LEDs"
- note removed: "SDC Relay Coil Driver"
- note removed: "TPS >0.9V"
- note removed: "Threshold Voltages (with max & min ranges) still need to be verified with sensor hardware"
- moved on the sheet: C1, C2, C6, C7, C8, C9, Q6, R1, R14, R15, R2, R24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
